Commit message: new changes

File: description/robot.urdf.xacro (robot description, xacro)
@@ -2,3 +2,4 @@
 <robot xmlns:xacro="http://www.ros.org/wiki/xacro"  name="robot">
     <xacro:include filename = "robot_core.xacro" />
+    <xacro:include filename = "gazebo_control.xacro"/>
 </robot>

File: description/robot_core.xacro (robot description, xacro)
@@ -32,5 +32,5 @@
     </visual>
     <collision>
-        <origin xyz = "0.15 0.0 0.075"/>
+        <origin xyz = "0.15 0 0.075"/>
         <geometry>
             <box size = "0.3 0.3 0.15"/>
@@ -38,7 +38,12 @@
     </collision>
     <xacro:inertial_box mass = "0.5" x = "0.3" y="0.3" z = "0.15">
-        <origin xyz = "0.15 0 0.75" rpy ="0 0 0 "/>
+        <origin xyz = "0.15 0 0.075" rpy ="0 0 0 "/>
     </xacro:inertial_box>
 </link>
+    <gazebo reference = "chassis">
+        <material>
+           Gazebo/White
+        </material>
+    </gazebo>
 <!-- LEFT WHEEL LINK -->
     <joint name = "left_wheel_joint" type = "continuous">
@@ -64,4 +69,9 @@
         </xacro:inertial_cylinder>
     </link>
+        <gazebo reference = "left_wheel">
+            <material>
+            Gazebo/Blue
+            </material>
+        </gazebo>
 <!-- RIGHT WHEEL LINK -->
     <joint name = "right_wheel_joint" type = "continuous">
@@ -87,4 +97,9 @@
         </xacro:inertial_cylinder>
     </link>
+        <gazebo reference = "right_wheel">
+            <material>
+            Gazebo/Blue
+            </material>
+        </gazebo>
     <!-- CASTER WHEEL LINK -->
      <joint name = "caster_wheel_joint" type = "fixed">
@@ -104,4 +119,5 @@
                 <sphere radius = "0.05"/>
             </geometry>
+            <material name = "black"/>
         </collision>
         <xacro:inertial_sphere mass = "0.1" radius="0.05">
@@ -109,3 +125,10 @@
         </xacro:inertial_sphere>
      </link>
+     <gazebo reference = "caster_wheel">
+            <material>
+            Gazebo/Black
+            </material>
+            <mu1 value="0.001"/>
+            <mu2 value = "0.001"/>
+        </gazebo>
 </robot>
